Commit message: update

File: description/urdf/robot_description.urdf (robot description, URDF)
Before this commit: robot robot_description, 21 links, 20 joints
Links:
- added link usb_cam_link
Joints:
- added joint usb_cam_joint: type fixed, parent base_link, child usb_cam_link, origin xyz=0.06 0 0.360 rpy=0 0 0, axis 1 1 1

Commit message: minor updates

File: description/urdf/robot_description.urdf (robot description, URDF)
Before this commit: robot robot_description, 22 links, 21 joints
Links:
- removed link lidar_link
- added link base_footprint
Joints:
- removed joint left_tread_joint
- removed joint right_tread_joint
- added joint base_to_footprint: type fixed, parent base_link, child base_footprint, origin xyz=0 0 0 rpy=0 0 0
- added joint left_tread: type continuous, parent base_link, child left_tread_link, origin xyz=-0.178 0.090 0 rpy=0 0 0, axis 1 1 0
- added joint right_tread: type continuous, parent base_link, child right_tread_link, origin xyz=-0.178 -0.090 0 rpy=0 0 0, axis 1 1 0
