Commit message: Code audit: fix build-blocking bugs, security leak, and add README
- Remove hardcoded GitHub token from update_repository.sh (security)
- Remove broken nxt_python package stub that failed catkin_make
- Add missing catkin_install_python declarations for python nodes
- Fix addDelta NameError in base_odometry.py (not exported by tf_conversions)
- Fix inverted odom/base_link TF frames in base_odometry.py
- Fix laser_scan_dir param type (bool vs string) in core.launch
- Fix lidar frame_id: use laser_link from URDF (base_laser was undefined)
- Disable imu_used in robot_pose_ekf (no imu_data published)
- Fix URDF: restore missing lidar_link, fix mesh path
- Fix int(msg.rotations) truncation in joint command conversion (4x)
- Fix emergency_shutdown: subscriber leak and uncancelable shutdown
- Fix update_full.sh calling removed update_filesystem.sh
- Fix rviz_core.launch pointing to nonexistent rviz config
- Add slam.launch (gmapping) and teleop_joy.launch for project goals
- Rewrite main README.md documenting hardware, setup, SLAM and AI layer

Co-authored-by: rodolphemds <rodolphemds@users.noreply.github.com>

File: description/urdf/robot_description.urdf (robot description, URDF)
Before this commit: robot robot_description, 22 links, 22 joints
Links:
- added link lidar_link
- link base_link: geometry collision box size=0.360 0.180 0.530; visual mesh filename=/betabot/description/meshes/robot_3d_model.dae

Commit message: Add measured URDF description and LEGO-derived meshes for BetaBot
- Dimensions derived from the BrickLink Studio model (meshes/lego model.io)
  using the LDraw scale (1 LDU = 0.4 mm), validated on Technic axles and
  official NXT part sizes. Assembled robot: 374 x 133 x 446 mm.
- generate_meshes.py extracts the LDraw model from the .io archive and builds
  per-link STL meshes (base, torso, head, arms, full) in ROS frames.
- Rewrote robot_description.urdf with the measured kinematic chain and all
  frames used by the existing ROS code, including the base_laser frame used
  by the ldlidar_stl driver (previously missing from the URDF).
- dimensions.json records the measured bounding box and joint origins.

Co-authored-by: rodolphemds <rodolphemds@users.noreply.github.com>

File: description/urdf/robot_description.urdf (robot description, URDF)
Before this commit: robot robot_description, 22 links, 22 joints
Links:
- removed link ambient_temperature_sensor_link
- removed link gps_link
- removed link magnetic_field_sensor_link
- removed link relative_humidity_sensor_link
- added link base_laser
- link arms_link: mass None -> 0.15; geometry collision box size=0.338 0.100 0.043; visual mesh filename=file:///betabot/description/meshes/betabot_arms.stl
- link base_link: mass 3 -> 3.0; geometry collision box size=0.374 0.133 0.160; visual mesh filename=file:///betabot/description/meshes/betabot_base.stl
- link head_link: mass None -> 0.2; geometry collision box size=0.272 0.111 0.092; visual mesh filename=file:///betabot/description/meshes/betabot_head.stl
- link laser_link: mass None -> 0.05; geometry collision cylinder length=0.036 radius=0.038; visual cylinder length=0.036 radius=0.038
- link left_tread_link: mass None -> 0.05; geometry collision cylinder length=0.133 radius=0.025
- link right_tread_link: mass None -> 0.05; geometry collision cylinder length=0.133 radius=0.025
- link torso_link: mass None -> 0.8; geometry collision box size=0.367 0.104 0.441; visual mesh filename=file:///betabot/description/meshes/betabot_torso.stl
Joints:
- removed joint ambient_temperature_sensor_joint
- removed joint gps_joint
- removed joint lidar_joint
- removed joint magnetic_field_sensor_joint
- removed joint relative_humidity_sensor_joint
- added joint laser_frame_joint: type fixed, parent laser_link, child base_laser, origin xyz=0 0 0.018 rpy=3.14159265359 0 0
- joint arms_joint: axis 1 1 1 -> 0 1 0; limit lower=-2.443 upper=4.363 effort=0.5 velocity=1 -> lower=-2.443 upper=4.363 effort=50 velocity=1.0; origin xyz=0.060 0 0.310 rpy=0 0 0 -> xyz=0.1786 0 0.154 rpy=0 0 0; parent base_link -> torso_link
- joint back_bumper_joint: axis 1 1 1 -> (none); origin xyz=0.180 0 0 rpy=0 0 0 -> xyz=-0.140 0 0.070 rpy=0 0 0
- joint base_to_footprint: origin xyz=0 0 0 rpy=0 0 0 -> xyz=0 0 -0.025 rpy=0 0 0
- joint color_sensor_joint: axis 1 1 1 -> (none); origin xyz=0.090 0.065 0.340 rpy=0 0 0 -> xyz=0.130 0 0.020 rpy=0 1.57079632679 0
- joint head_joint: axis 1 1 0 -> 0 0 1; limit lower=-7.156 upper=7.156 effort=0.75 velocity=1 -> lower=-7.156 upper=7.156 effort=50 velocity=1.0; origin xyz=-0.060 0 -0.360 rpy=0 0 0 -> xyz=0.0362 0 0.122 rpy=0 0 0; parent base_link -> torso_link
- joint imu_joint: axis 1 1 1 -> (none); origin xyz=0 0 0 rpy=0 0 -1.57079632679 -> xyz=-0.050 0 0.080 rpy=0 0 -1.57079632679
- joint laser_joint: axis 1 1 1 -> 0 0 1; limit lower=0.0 upper=1.658 effort=0.5 velocity=1 -> lower=-0.3 upper=2.0 effort=50 velocity=1.0; origin xyz=0.090 0.065 0.250 rpy=0 0 0 -> xyz=0 0 0.0716 rpy=0 0 0; parent base_link -> head_link
- joint left_bumper_joint: axis 1 1 1 -> (none); origin xyz=-0.180 0.090 0 rpy=0 0 0 -> xyz=0.140 0.045 0.070 rpy=0 0 0
- joint left_tread: axis 1 1 0 -> 0 1 0; origin xyz=-0.178 0.090 0 rpy=0 0 0 -> xyz=0 0.0665 0 rpy=0 1.57079632679 0
- joint line_following_sensor_joint: axis 1 1 1 -> (none); origin xyz=-0.140 0 0 rpy=0 0 0 -> xyz=0.120 0 0.010 rpy=0 1.57079632679 0
- joint rfid_sensor_joint: axis 1 1 1 -> (none); origin xyz=0 -0.5 0.170 rpy=0 0 0 -> xyz=-0.050 0 0.100 rpy=0 0 0
- joint right_bumper_joint: axis 1 1 1 -> (none); origin xyz=-0.180 -0.090 0 rpy=0 0 0 -> xyz=0.140 -0.045 0.070 rpy=0 0 0
- joint right_tread: axis 1 1 0 -> 0 1 0; origin xyz=-0.178 -0.090 0 rpy=0 0 0 -> xyz=0 -0.0665 0 rpy=0 1.57079632679 0
- joint sound_sensor_joint: axis 1 1 1 -> (none); origin xyz=0.06 0.50 0.280 rpy=0 0 0 -> xyz=0 0 0.046 rpy=0 0 0; parent base_link -> head_link
- joint torso_joint: axis 1 1 1 -> 0 0 1; limit lower=0.0 upper=16.581 effort=1 velocity=1 -> lower=-2.967 upper=2.967 effort=50 velocity=1.0; origin xyz=0.060 0 0.150 rpy=0 0 0 -> xyz=0.0096 0 0.1824 rpy=0 0 0
- joint ultrasonic_sensor_joint: axis 1 1 1 -> (none); origin xyz=0.06 0 0.360 rpy=0 0 0 -> xyz=0.072 0 0.010 rpy=0 0 0; parent base_link -> head_link
- joint usb_cam_joint: axis 1 1 1 -> (none); origin xyz=0.06 0 0.360 rpy=0 0 0 -> xyz=0.09 0 0.055 rpy=0 0 0; parent base_link -> head_link

Commit message: Replace LDraw draft with Polycam scan-based description
- meshes: segment betabot_scan.glb (LiDAR photogrammetry, metric scale)
  into base/torso/arms/head STLs in ROS conventions (X fwd, Y left, Z up),
  anchored on joint origins; scan axes mapping X=-Z_scan, Y=-X_scan, Z=Y_scan
- dimensions: 417 x 273 x 486 mm, scale validated on NXT brick (108.4 mm)
  and tread_radius 0.025 m
- URDF: joint origins and collision boxes updated from scan measurements
- generate_meshes.py: regenerates STLs + dimensions.json from the GLB
  (pure stdlib); lego model.io kept as reference only

Co-authored-by: rodolphemds <rodolphemds@users.noreply.github.com>

File: description/urdf/robot_description.urdf (robot description, URDF)
Before this commit: robot betabot, 19 links, 18 joints
Links:
- link arms_link: geometry collision box size=0.298 0.242 0.107; visual mesh filename=file:///betabot/description/meshes/betabot_arms.stl
- link base_link: geometry collision box size=0.417 0.245 0.135; visual mesh filename=file:///betabot/description/meshes/betabot_base.stl
- link head_link: geometry collision box size=0.115 0.100 0.130; visual mesh filename=file:///betabot/description/meshes/betabot_head.stl
- link torso_link: geometry collision box size=0.242 0.187 0.138; visual mesh filename=file:///betabot/description/meshes/betabot_torso.stl
Joints:
- joint arms_joint: origin xyz=0.1786 0 0.154 rpy=0 0 0 -> xyz=0 0 0.078 rpy=0 0 0
- joint back_bumper_joint: origin xyz=-0.140 0 0.070 rpy=0 0 0 -> xyz=-0.185 0 0.070 rpy=0 0 0
- joint color_sensor_joint: origin xyz=0.130 0 0.020 rpy=0 1.57079632679 0 -> xyz=0.160 0 0.020 rpy=0 1.57079632679 0
- joint head_joint: origin xyz=0.0362 0 0.122 rpy=0 0 0 -> xyz=0 0 0.149 rpy=0 0 0
- joint imu_joint: origin xyz=-0.050 0 0.080 rpy=0 0 -1.57079632679 -> xyz=-0.100 0 0.080 rpy=0 0 -1.57079632679
- joint laser_joint: origin xyz=0 0 0.0716 rpy=0 0 0 -> xyz=0 0 0.130 rpy=0 0 0
- joint left_bumper_joint: origin xyz=0.140 0.045 0.070 rpy=0 0 0 -> xyz=0.185 0.045 0.070 rpy=0 0 0
- joint line_following_sensor_joint: origin xyz=0.120 0 0.010 rpy=0 1.57079632679 0 -> xyz=0.150 0 0.010 rpy=0 1.57079632679 0
- joint rfid_sensor_joint: origin xyz=-0.050 0 0.100 rpy=0 0 0 -> xyz=-0.100 0 0.100 rpy=0 0 0
- joint right_bumper_joint: origin xyz=0.140 -0.045 0.070 rpy=0 0 0 -> xyz=0.185 -0.045 0.070 rpy=0 0 0
- joint sound_sensor_joint: origin xyz=0 0 0.046 rpy=0 0 0 -> xyz=0 0 0.100 rpy=0 0 0
- joint torso_joint: origin xyz=0.0096 0 0.1824 rpy=0 0 0 -> xyz=0 0 0.182 rpy=0 0 0
- joint ultrasonic_sensor_joint: origin xyz=0.072 0 0.010 rpy=0 0 0 -> xyz=0.115 0 0.065 rpy=0 0 0
- joint usb_cam_joint: origin xyz=0.09 0 0.055 rpy=0 0 0 -> xyz=0.09 0 0.065 rpy=0 0 0
